Commit message: Docker Noetic run + Quest3S grip deadman

File: src/Piper_ros/src/piper_description/urdf/piper_description.urdf (robot description, URDF)
Before this commit: robot piper_description, 10 links, 9 joints
Links:
- link base_link: geometry collision mesh filename=/ws/src/Piper_ros/src/piper_description/meshes/base_link.STL; visual mesh filename=/ws/src/Piper_ros/src/piper_description/meshes/base_link.STL
- link gripper_base: geometry collision mesh filename=/ws/src/Piper_ros/src/piper_description/meshes/gripper_base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; visual mesh filename=/ws/src/Piper_ros/src/piper_description/meshes/gripper_base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
- link link1: geometry collision mesh filename=/ws/src/Piper_ros/src/piper_description/meshes/link1.STL; visual mesh filename=/ws/src/Piper_ros/src/piper_description/meshes/link1.STL
- link link2: geometry collision mesh filename=/ws/src/Piper_ros/src/piper_description/meshes/link2.STL; visual mesh filename=/ws/src/Piper_ros/src/piper_description/meshes/link2.STL
- link link3: geometry collision mesh filename=/ws/src/Piper_ros/src/piper_description/meshes/link3.STL; visual mesh filename=/ws/src/Piper_ros/src/piper_description/meshes/link3.STL
- link link4: geometry collision mesh filename=/ws/src/Piper_ros/src/piper_description/meshes/link4.STL; visual mesh filename=/ws/src/Piper_ros/src/piper_description/meshes/link4.STL
- link link5: geometry collision mesh filename=/ws/src/Piper_ros/src/piper_description/meshes/link5.STL; visual mesh filename=/ws/src/Piper_ros/src/piper_description/meshes/link5.STL
- link link6: geometry collision mesh filename=/ws/src/Piper_ros/src/piper_description/meshes/link6.STL; visual mesh filename=/ws/src/Piper_ros/src/piper_description/meshes/link6.STL
- link link7: geometry collision mesh filename=/ws/src/Piper_ros/src/piper_description/meshes/link7.STL; visual mesh filename=/ws/src/Piper_ros/src/piper_description/meshes/link7.STL
- link link8: geometry collision mesh filename=/ws/src/Piper_ros/src/piper_description/meshes/link8.STL; visual mesh filename=/ws/src/Piper_ros/src/piper_description/meshes/link8.STL
